File: Solenoid_Valve-fin.kicad_pcb (KiCad board)
At the start: 2 copper layers, 90 x 100 mm, 124 parts, among them IC1 Si8621AB-B-ISR, J1 Conn_01x02, J10 Conn_01x02, J11 Conn_01x02, J12 Conn_01x02, J13 Conn_01x02, J14 Conn_01x02, J15 Conn_01x02, J16 Conn_01x02, J17 Conn_01x02, J18 Conn_01x02, J19 Conn_01x02, J2 Conn_01x05, J20 Conn_01x02, J21 Bus_PCIexpress_x1_36_Position, J3 Conn_01x02, J4 Conn_01x02, J5 Conn_01x02, J6 Conn_01x02, J8 Conn_01x02, J9 Conn_01x02, Q1 ULN2004D1013TR, Q2 ULN2004D1013TR, Q3 ULN2004D1013TR, SW1 SW_Push, U1 LDO_3.3V, U2 STM32F042K6Tx, U3 MCP2562-E-SN, U4 L7812, U5 LDL1117S33R

Commit message: change
Remove NRST SW
clean
Changed lines of the file:
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@@
-(kicad_pcb (version 20171130) (host pcbnew "(5.1.4)-1")
+(kicad_pcb (version 20171130) (host pcbnew "(5.1.5)-3")
   (general
     (thickness 1.6)
     (drawings 54)
-    (tracks 1796)
+    (tracks 1795)
     (zones 0)
     (modules 124)
@@
   (via (at 174.47 100.65) (size 0.6) (drill 0.3) (layers F.Cu B.Cu) (net 4))
   (via (at 165.58 100.65) (size 0.6) (drill 0.3) (layers F.Cu B.Cu) (net 4))
-  (segment (start 139.404 108.267) (end 139.5 108.17) (width 0.25) (layer B.Cu) (net 4))
   (segment (start 129.5 99.425) (end 129.5 98.325) (width 0.25) (layer F.Cu) (net 4) (status 10))
   (via (at 207.5 117.5) (size 0.6) (drill 0.3) (layers F.Cu B.Cu) (net 4))

Commit message: Prototype-1.1
Parts:
- removed C3 (x2): 0.1uF, Capacitor_SMD:C_0805_2012Metric
- removed the J1 at (189.0, 76.0)
- removed the J1 at (141.0, 84.0)
- removed J21 (x2): Bus_PCIexpress_x1_36_Position, library:BUS_PCIexpress_x1_36_Position
- removed R3 (x2): 10K, Resistor_SMD:R_0603_1608Metric
- removed SW1 (x2): SW_Push, SamacSys_Parts:PTS647SM38SMTR2LFS
- removed the U1 at (205.4, 52.5)
- removed the U1 at (124.6, 107.5)
- added J1: Bus_mechaken_PCIexpress_x16_164_Position, PCIe:BUS_mechaken_PCIexpress_x16_164_Position, F.Cu at (121.0, 76.0)
- added J1: Bus_mechaken_PCIexpress_x16_164_Position, PCIe:BUS_mechaken_PCIexpress_x16_164_Position, F.Cu at (121.0, 126.0)
- added J7: Conn_01x03, Connector_JST:JST_XH_B3B-XH-A_1x03_P2.50mm_Vertical, F.Cu at (142.7, 34.1)
- added J7: Conn_01x03, Connector_JST:JST_XH_B3B-XH-A_1x03_P2.50mm_Vertical, F.Cu at (142.7, 84.1)
- added U1: LDL1117S33R, Package_TO_SOT_SMD:SOT-223-3_TabPin2, F.Cu at (126.5, 58.6)
- added U1: LDL1117S33R, Package_TO_SOT_SMD:SOT-223-3_TabPin2, F.Cu at (126.5, 108.7)
- C1 (x2): value 0.1uF -> 1.0uF
- C2 (x2): value 0.1uF -> 4.7uF
- moved J2 93.0 mm to (123.0, 34.0), turned to 0 degrees
- moved R2 92.8 mm to (121.0, 40.2), turned to 270 degrees
- moved D1 87.1 mm to (121.8, 49.5), turned to 90 degrees
- moved C1 85.7 mm to (123.2, 64.7), turned to 0 degrees
- moved J11 85.6 mm to (203.7, 36.7), turned to 90 degrees
- moved D10 84.5 mm to (201.4, 43.5), turned to 180 degrees
- moved R1 82.0 mm to (124.9, 49.5), turned to 90 degrees
- moved C5 81.2 mm to (126.7, 68.5), turned to 0 degrees
- moved D16 79.1 mm to (201.6, 59.9), turned to 180 degrees
- moved J17 77.6 mm to (203.7, 51.9), turned to 90 degrees
- moved C2 77.0 mm to (127.7, 64.7), turned to 180 degrees
- moved U2 77.0 mm to (127.9, 44.7), turned to 225 degrees
- moved D11 76.9 mm to (198.6, 36.3), turned to 90 degrees
- moved C4 75.7 mm to (127.2, 52.6), turned to 180 degrees
- moved IC1 73.5 mm to (128.3, 57.3), turned to 180 degrees
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Connections:
- C1 pad 1: (no net) -> +5V
- C1 pad 2: (no net) -> GND
- C10 pad 1: (no net) -> 3.3V
- C10 pad 2: (no net) -> GNDPWR
- C2 pad 1: (no net) -> GND
- C2 pad 2: (no net) -> +3V3
- C4 pad 1: (no net) -> GNDPWR
- C4 pad 2: (no net) -> 3.3V
- C5 pad 1: (no net) -> GND
- C5 pad 2: (no net) -> +3V3
- C6 pad 1: (no net) -> GND
- C6 pad 2: (no net) -> +5V
- C7 pad 1: (no net) -> VCC
- C7 pad 2: (no net) -> GNDPWR
- C8 pad 1: (no net) -> +12V
- C8 pad 2: (no net) -> GNDPWR
- C9 pad 1: (no net) -> +12V
- C9 pad 2: (no net) -> GNDPWR
- D1 pad 1: (no net) -> GNDPWR
- D1 pad 2: (no net) -> Net-(D1-Pad2)
- D10 pad 1: (no net) -> +12V
- D10 pad 2: (no net) -> Solenoid_B1
- D11 pad 1: (no net) -> +12V
- D11 pad 2: (no net) -> Solenoid_B2
- D12 pad 1: (no net) -> +12V
- D12 pad 2: (no net) -> Solenoid_B3
- D13 pad 1: (no net) -> +12V
- D13 pad 2: (no net) -> Solenoid_B4
- D14 pad 1: (no net) -> +12V
- D14 pad 2: (no net) -> Solenoid_A5
- D15 pad 1: (no net) -> +12V
- D15 pad 2: (no net) -> Solenoid_A6
- D16 pad 1: (no net) -> +12V
- D16 pad 2: (no net) -> Solenoid_A7
- D17 pad 1: (no net) -> +12V
- D17 pad 2: (no net) -> Solenoid_B5
- D18 pad 1: (no net) -> +12V
- D18 pad 2: (no net) -> Solenoid_B6
- D19 pad 1: (no net) -> +12V
- D19 pad 2: (no net) -> Solenoid_B7
- D2 pad 1: (no net) -> +12V
- D2 pad 2: (no net) -> Solenoid_C1
- D3 pad 1: (no net) -> +12V
- D3 pad 2: (no net) -> Solenoid_C2
- D4 pad 1: (no net) -> +12V
- D4 pad 2: (no net) -> Solenoid_C3
- D6 pad 1: (no net) -> +12V
- D6 pad 2: (no net) -> Solenoid_A1
- D7 pad 1: (no net) -> +12V
- D7 pad 2: (no net) -> Solenoid_A2
- D8 pad 1: (no net) -> +12V
- D8 pad 2: (no net) -> Solenoid_A3
- D9 pad 1: (no net) -> +12V
- D9 pad 2: (no net) -> Solenoid_A4
- IC1 pad 1: (no net) -> +3V3
- IC1 pad 2: (no net) -> CAN_RXD
- IC1 pad 3: (no net) -> CAN_TXD
- IC1 pad 4: (no net) -> GND
- IC1 pad 5: (no net) -> GNDPWR
- IC1 pad 6: (no net) -> CAN_TD
- IC1 pad 7: (no net) -> CAN_RD
- IC1 pad 8: (no net) -> 3.3V
- J10 pad 1: (no net) -> +12V
- J10 pad 2: (no net) -> Solenoid_A4
- J11 pad 1: (no net) -> +12V
- J11 pad 2: (no net) -> Solenoid_B1
- J12 pad 1: (no net) -> +12V
- J12 pad 2: (no net) -> Solenoid_B2
- J13 pad 1: (no net) -> +12V
- J13 pad 2: (no net) -> Solenoid_B3
- J14 pad 1: (no net) -> +12V
- J14 pad 2: (no net) -> Solenoid_B4
- J15 pad 1: (no net) -> +12V
- J15 pad 2: (no net) -> Solenoid_A5
- J16 pad 1: (no net) -> +12V
- J16 pad 2: (no net) -> Solenoid_A6
- J17 pad 1: (no net) -> +12V
- J17 pad 2: (no net) -> Solenoid_A7
- J18 pad 1: (no net) -> +12V
- J18 pad 2: (no net) -> Solenoid_B5
- J19 pad 1: (no net) -> +12V
- J19 pad 2: (no net) -> Solenoid_B6
- J2 pad 1: (no net) -> 3.3V
- J2 pad 2: (no net) -> /SWCLK
- J2 pad 3: (no net) -> GNDPWR
- J2 pad 4: (no net) -> /SWDIO
- J2 pad 5: (no net) -> NRST
- J2 pad 2: GNDPWR -> /SWCLK
- J2 pad 3: /SWCLK -> GNDPWR
- J20 pad 1: (no net) -> +12V
- J20 pad 2: (no net) -> Solenoid_B7
- J3 pad 1: (no net) -> +12V
- J3 pad 2: (no net) -> Solenoid_A2
- J4 pad 1: (no net) -> +12V
- J4 pad 2: (no net) -> Solenoid_C1
- J5 pad 1: (no net) -> +12V
- J5 pad 2: (no net) -> Solenoid_C2
- J6 pad 1: (no net) -> +12V
- J6 pad 2: (no net) -> Solenoid_C3
- J8 pad 1: (no net) -> +12V
- J8 pad 2: (no net) -> Solenoid_A1
- J9 pad 1: (no net) -> +12V
- J9 pad 2: (no net) -> Solenoid_A3
- Q1 pad 1: (no net) -> IC_A1
- Q1 pad 10: (no net) -> Solenoid_A7
- Q1 pad 11: (no net) -> Solenoid_A6
- Q1 pad 12: (no net) -> Solenoid_A5
- Q1 pad 13: (no net) -> Solenoid_A4
- Q1 pad 14: (no net) -> Solenoid_A3
- Q1 pad 15: (no net) -> Solenoid_A2
- Q1 pad 16: (no net) -> Solenoid_A1
- Q1 pad 2: (no net) -> IC_A2
- Q1 pad 3: (no net) -> IC_A3
- Q1 pad 4: (no net) -> IC_A4
- Q1 pad 5: (no net) -> IC_A5
- Q1 pad 6: (no net) -> IC_A6
- Q1 pad 7: (no net) -> IC_A7
- Q1 pad 8: (no net) -> GNDPWR
- Q1 pad 9: (no net) -> +12V
- Q2 pad 1: (no net) -> IC_B1
- Q2 pad 10: (no net) -> Solenoid_B7
- Q2 pad 11: (no net) -> Solenoid_B6
- Q2 pad 12: (no net) -> Solenoid_B5
- Q2 pad 13: (no net) -> Solenoid_B4
- Q2 pad 14: (no net) -> Solenoid_B3
- Q2 pad 15: (no net) -> Solenoid_B2
- Q2 pad 16: (no net) -> Solenoid_B1
- Q2 pad 2: (no net) -> IC_B2
- Q2 pad 3: (no net) -> IC_B3
- Q2 pad 4: (no net) -> IC_B4
- Q2 pad 5: (no net) -> IC_B5
- Q2 pad 6: (no net) -> IC_B6
- Q2 pad 7: (no net) -> IC_B7
- Q2 pad 8: (no net) -> GNDPWR
- Q2 pad 9: (no net) -> +12V
- Q3 pad 1: (no net) -> IC_C1
- Q3 pad 14: (no net) -> Solenoid_C3
- Q3 pad 15: (no net) -> Solenoid_C2
- Q3 pad 16: (no net) -> Solenoid_C1
- Q3 pad 2: (no net) -> IC_C2
- Q3 pad 3: (no net) -> IC_C3
- Q3 pad 8: (no net) -> GNDPWR
- Q3 pad 9: (no net) -> +12V
- R1 pad 1: (no net) -> +3V3
- R1 pad 2: (no net) -> Net-(D1-Pad2)
- R2 pad 1: (no net) -> /BOOT
- R2 pad 2: (no net) -> +3V3
- S1 pad 3: (no net) -> DIP_SW_1 (x2)
- S1 pad 4: (no net) -> DIP_SW_2 (x2)
- S1 pad 5: (no net) -> 3.3V
- S1 pad 6: (no net) -> 3.3V
- S1 pad 7: (no net) -> 3.3V
- S1 pad 8: (no net) -> 3.3V
- S1 pad 1: DIP_SW_1 -> (no net)
- S1 pad 2: DIP_SW_2 -> (no net)
- U2 pad 1: (no net) -> 3.3V
- U2 pad 10: (no net) -> IC_A6
- U2 pad 11: (no net) -> IC_A5
- U2 pad 12: (no net) -> IC_A4
- U2 pad 13: (no net) -> IC_A3
- U2 pad 14: (no net) -> IC_A2
- U2 pad 15: (no net) -> IC_A1
- U2 pad 16: (no net) -> GNDPWR
- U2 pad 17: (no net) -> 3.3V
- U2 pad 18: (no net) -> IC_C3
- U2 pad 19: (no net) -> IC_C2
- U2 pad 2: (no net) -> IC_B7
- U2 pad 20: (no net) -> IC_C1
- U2 pad 21: (no net) -> CAN_RD
- U2 pad 22: (no net) -> CAN_TD
- U2 pad 23: (no net) -> /SWDIO
- U2 pad 24: (no net) -> /SWCLK
- U2 pad 25: (no net) -> VCP_RX
- U2 pad 26: (no net) -> IC_B1
- U2 pad 27: (no net) -> IC_B2
- U2 pad 28: (no net) -> IC_B3
- U2 pad 29: (no net) -> DIP_SW_1
- U2 pad 3: (no net) -> IC_B6
- U2 pad 30: (no net) -> DIP_SW_2
- U2 pad 31: (no net) -> /BOOT
- U2 pad 32: (no net) -> GNDPWR
- U2 pad 4: (no net) -> NRST
- U2 pad 5: (no net) -> 3.3V
- U2 pad 6: (no net) -> IC_B5
- U2 pad 7: (no net) -> IC_B4
- U2 pad 8: (no net) -> VCP_TX
- U2 pad 9: (no net) -> IC_A7
- U3 pad 1: (no net) -> CAN_TXD
- U3 pad 2: (no net) -> GND
- U3 pad 3: (no net) -> +5V
- U3 pad 4: (no net) -> CAN_RXD
- U3 pad 5: (no net) -> +3V3
- U3 pad 6: (no net) -> CAN-
- U3 pad 7: (no net) -> CAN+
- U3 pad 8: (no net) -> GND
- U4 pad 1: (no net) -> VCC
- U4 pad 2: (no net) -> GNDPWR
- U4 pad 3: (no net) -> +12V
- U5 pad 1: (no net) -> GNDPWR
- U5 pad 2: (no net) -> 3.3V
- U5 pad 3: (no net) -> +12V
Routing:
- net (no net): track 1998.3 -> 0.00 mm, vias 100 -> 0
- net +12V: track 334.0 -> 733.2 mm
- net +3V3: track 67.1 -> 164.7 mm, vias 2 -> 4
- net Solenoid_B1: track 70.1 -> 148.5 mm
- net 3.3V: track 95.6 -> 168.2 mm
- net Solenoid_A7: track 69.7 -> 141.4 mm
- net Solenoid_A6: track 65.2 -> 130.5 mm, vias 5 -> 10
- net Solenoid_A5: track 64.0 -> 127.4 mm
- net Solenoid_B2: track 60.2 -> 118.9 mm
- net Net-(J1-PadB9): track 0.00 -> 58.0 mm
- net +5V: track 64.9 -> 117.1 mm, vias 2 -> 4
- net Solenoid_B3: track 50.0 -> 100.0 mm
- net Solenoid_C1: track 47.5 -> 97.0 mm
- net Solenoid_A4: track 48.4 -> 96.9 mm
- net IC_B1: track 48.0 -> 94.8 mm
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- removed copper zone on B.Cu, net (none)
- removed copper zone on F.Cu, net (none)
Other:
- board size 90 x 100 mm -> 85.9 x 100 mm
- board text added: "+3V3"
- board text added: "CAN Solenoid Driver x17 Prototype 1.1 Designed by TNK."
- board text added: "GND"
- board text added: "NRST"
- board text added: "SWCLK"
- board text added: "SWDIO"
- board text added: "VCP_TX"
- board text added: "VXP_TX"
- board text removed: "CAN Solenoid Valve x17 Prototype 1.0 Designed by TNK."

Commit message: Release
ガーバーファイルを出力
Parts:
- removed C10: 4.7uF, Capacitor_SMD:C_0805_2012Metric
- removed the D1 at (121.8, 49.5)
- removed the D1 at (121.8, 99.5)
- removed the D18 at (163.0, 36.3)
- removed D19: D, Diode_SMD:D_2010_5025Metric
- removed the R1 at (124.9, 49.5)
- removed the R1 at (124.9, 99.5)
- removed R2: 10K, Resistor_SMD:R_0603_1608Metric
- added C3: 4.7uF, Capacitor_SMD:C_0805_2012Metric_Pad1.15x1.40mm_HandSolder, F.Cu at (203.4, 45.3)
- added D1: D, Diode_SMD:D_2010_5025Metric_Pad1.52x2.65mm_HandSolder, B.Cu at (143.9, 45.8)
- added D18: D_Schottky, Diode_SMD:D_0603_1608Metric_Pad1.05x0.95mm_HandSolder, B.Cu at (184.5, 40.5)
- added D18: D_Schottky, Diode_SMD:D_0603_1608Metric_Pad1.05x0.95mm_HandSolder, B.Cu at (151.6, 119.5)
- added D5: D, Diode_SMD:D_2010_5025Metric_Pad1.52x2.65mm_HandSolder, B.Cu at (168.1, 58.5)
- added R1: 10K, Resistor_SMD:R_0603_1608Metric_Pad1.05x0.95mm_HandSolder, B.Cu at (209.8, 69.9)
- C1: value 1.0uF -> 0.1uF; footprint Capacitor_SMD:C_0805_2012Metric -> Capacitor_SMD:C_0805_2012Metric_Pad1.15x1.40mm_HandSolder; moved to B.Cu
- C1: renamed from C5; footprint Capacitor_SMD:C_0805_2012Metric -> Capacitor_SMD:C_0805_2012Metric_Pad1.15x1.40mm_HandSolder
- C2: value 4.7uF -> 1.0uF; footprint Capacitor_SMD:C_0805_2012Metric -> Capacitor_SMD:C_0805_2012Metric_Pad1.15x1.40mm_HandSolder
- C2: renamed from C1; footprint Capacitor_SMD:C_0805_2012Metric -> Capacitor_SMD:C_0805_2012Metric_Pad1.15x1.40mm_HandSolder
- C3: renamed from C2; footprint Capacitor_SMD:C_0805_2012Metric -> Capacitor_SMD:C_0805_2012Metric_Pad1.15x1.40mm_HandSolder
- C4, C6: footprint Capacitor_SMD:C_0805_2012Metric -> Capacitor_SMD:C_0805_2012Metric_Pad1.15x1.40mm_HandSolder
- C4: renamed from C6; footprint Capacitor_SMD:C_0805_2012Metric -> Capacitor_SMD:C_0805_2012Metric_Pad1.15x1.40mm_HandSolder
- C5: value 0.1uF -> 1.0uF; footprint Capacitor_SMD:C_0805_2012Metric -> Capacitor_SMD:C_0805_2012Metric_Pad1.15x1.40mm_HandSolder
- C5: renamed from C9; footprint Capacitor_SMD:C_0805_2012Metric -> Capacitor_SMD:C_0805_2012Metric_Pad1.15x1.40mm_HandSolder
- C6: renamed from C4; footprint Capacitor_SMD:C_0805_2012Metric -> Capacitor_SMD:C_0805_2012Metric_Pad1.15x1.40mm_HandSolder
- C7: value 1uF -> 4.7uF
- C7: renamed from C10; footprint Capacitor_SMD:C_0805_2012Metric -> Capacitor_SMD:C_0805_2012Metric_Pad1.15x1.40mm_HandSolder
- C8: value 4.7uF -> 0.33uF; footprint Capacitor_SMD:C_0805_2012Metric -> Capacitor_SMD:C_0805_2012Metric_Pad1.15x1.40mm_HandSolder
- C8: renamed from C7; value 1uF -> 0.33uF
- C9: value 1.0uF -> 0.1uF; footprint Capacitor_SMD:C_0805_2012Metric -> Capacitor_SMD:C_0805_2012Metric_Pad1.15x1.40mm_HandSolder
- C9: renamed from C8; value 4.7uF -> 0.1uF; footprint Capacitor_SMD:C_0805_2012Metric -> Capacitor_SMD:C_0805_2012Metric_Pad1.15x1.40mm_HandSolder
- D1: renamed from D2; footprint Diode_SMD:D_2010_5025Metric -> Diode_SMD:D_2010_5025Metric_Pad1.52x2.65mm_HandSolder
- D10, D11, D12, D13, D14, D15, D16, D17, D2, D3, D4, D6, D7, D8, D9: footprint Diode_SMD:D_2010_5025Metric -> Diode_SMD:D_2010_5025Metric_Pad1.52x2.65mm_HandSolder
- D10: renamed from D12; footprint Diode_SMD:D_2010_5025Metric -> Diode_SMD:D_2010_5025Metric_Pad1.52x2.65mm_HandSolder
- D11: renamed from D13; footprint Diode_SMD:D_2010_5025Metric -> Diode_SMD:D_2010_5025Metric_Pad1.52x2.65mm_HandSolder
- D12: renamed from D14; footprint Diode_SMD:D_2010_5025Metric -> Diode_SMD:D_2010_5025Metric_Pad1.52x2.65mm_HandSolder
- D13: renamed from D15; footprint Diode_SMD:D_2010_5025Metric -> Diode_SMD:D_2010_5025Metric_Pad1.52x2.65mm_HandSolder
- D14: renamed from D16; footprint Diode_SMD:D_2010_5025Metric -> Diode_SMD:D_2010_5025Metric_Pad1.52x2.65mm_HandSolder
- D15: renamed from D17; footprint Diode_SMD:D_2010_5025Metric -> Diode_SMD:D_2010_5025Metric_Pad1.52x2.65mm_HandSolder
- D16: renamed from D18; footprint Diode_SMD:D_2010_5025Metric -> Diode_SMD:D_2010_5025Metric_Pad1.52x2.65mm_HandSolder
- D17: renamed from D19; footprint Diode_SMD:D_2010_5025Metric -> Diode_SMD:D_2010_5025Metric_Pad1.52x2.65mm_HandSolder
- D2: renamed from D3; footprint Diode_SMD:D_2010_5025Metric -> Diode_SMD:D_2010_5025Metric_Pad1.52x2.65mm_HandSolder
- D3: renamed from D4; footprint Diode_SMD:D_2010_5025Metric -> Diode_SMD:D_2010_5025Metric_Pad1.52x2.65mm_HandSolder
- D4: renamed from D6; footprint Diode_SMD:D_2010_5025Metric -> Diode_SMD:D_2010_5025Metric_Pad1.52x2.65mm_HandSolder
- D5: renamed from D7; footprint Diode_SMD:D_2010_5025Metric -> Diode_SMD:D_2010_5025Metric_Pad1.52x2.65mm_HandSolder
- D6: renamed from D8; footprint Diode_SMD:D_2010_5025Metric -> Diode_SMD:D_2010_5025Metric_Pad1.52x2.65mm_HandSolder
- D7: renamed from D9; footprint Diode_SMD:D_2010_5025Metric -> Diode_SMD:D_2010_5025Metric_Pad1.52x2.65mm_HandSolder
- D8: renamed from D10; footprint Diode_SMD:D_2010_5025Metric -> Diode_SMD:D_2010_5025Metric_Pad1.52x2.65mm_HandSolder
- D9: renamed from D11; footprint Diode_SMD:D_2010_5025Metric -> Diode_SMD:D_2010_5025Metric_Pad1.52x2.65mm_HandSolder
- J1 (x2): footprint PCIe:BUS_mechaken_PCIexpress_x16_164_Position -> PCIe:BUS_mechaken_PCIexpress_x16
- J2: value Conn_01x05 -> Conn_01x02; footprint Connector_JST:JST_XH_B5B-XH-A_1x05_P2.50mm_Vertical -> Connector_JST:JST_XH_B2B-XH-A_1x02_P2.50mm_Vertical; moved to F.Cu
- J4: value Conn_01x02 -> Conn_01x03; footprint Connector_JST:JST_XH_B2B-XH-A_1x02_P2.50mm_Vertical -> Connector_JST:JST_XH_B3B-XH-A_1x03_P2.50mm_Vertical
- J5: value Conn_01x02 -> Conn_01x05; footprint Connector_JST:JST_XH_B2B-XH-A_1x02_P2.50mm_Vertical -> Connector_JST:JST_XH_B5B-XH-A_1x05_P2.50mm_Vertical; moved to B.Cu
- J7: value Conn_01x03 -> Conn_01x02; footprint Connector_JST:JST_XH_B3B-XH-A_1x03_P2.50mm_Vertical -> Connector_JST:JST_XH_B2B-XH-A_1x02_P2.50mm_Vertical
- R1: renamed from R2; footprint Resistor_SMD:R_0603_1608Metric -> Resistor_SMD:R_0603_1608Metric_Pad1.05x0.95mm_HandSolder
- U2: value STM32F042K6Tx -> MCP2562-E-SN; footprint Package_QFP:LQFP-32_7x7mm_P0.8mm -> Package_SO:SOIC-8_3.9x4.9mm_P1.27mm
- U3: value MCP2562-E-SN -> STM32F042K6Tx; footprint Package_SO:SOIC-8_3.9x4.9mm_P1.27mm -> Package_QFP:LQFP-32_7x7mm_P0.8mm
- U4: value L7812 -> LDL1117S33R; footprint Package_TO_SOT_SMD:TO-252-2 -> Package_TO_SOT_SMD:SOT-223-3_TabPin2
- U5: value LDL1117S33R -> NJM7812; footprint Package_TO_SOT_SMD:SOT-223-3_TabPin2 -> Package_TO_SOT_SMD:TO-252-2
- U5: renamed from U4; value L7812 -> NJM7812
- moved J1 98.5 mm to (210.1, 34.0), turned to 180 degrees
- moved J11 84.6 mm to (127.4, 73.3), turned to 270 degrees
- moved C1 84.2 mm to (204.2, 41.5), turned to 180 degrees
- moved C2 82.4 mm to (207.9, 45.3)
- moved U1 78.3 mm to (204.6, 51.4), turned to 180 degrees
- moved J17 76.5 mm to (127.4, 58.1), turned to 270 degrees
- moved IC1 74.6 mm to (202.8, 52.7), turned to 0 degrees
- moved U3 73.1 mm to (203.2, 65.3), turned to 45 degrees
- moved U2 73.1 mm to (201.0, 45.7), turned to 0 degrees
- moved J12 69.0 mm to (136.3, 73.3), turned to 270 degrees
- moved C4 68.8 mm to (195.7, 45.9), turned to 90 degrees
- moved C6 68.8 mm to (203.9, 57.4), turned to 0 degrees
- moved D10 67.2 mm to (141.4, 73.7), turned to 270 degrees
- moved C5 61.3 mm to (184.9, 49.2), turned to 270 degrees
- moved D14 60.2 mm to (129.6, 50.7), turned to 0 degrees
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- renumbered J4 to J2, J5 to J3, J7 to J4, J2 to J5, J8 to J7, J3 to J8, U3 to U2, U2 to U3, U5 to U4
Connections:
- C1 pad 1: +5V -> GND
- C1 pad 2: GND -> +3V3
- C2 pad 1: GND -> +5V
- C2 pad 2: +3V3 -> GND
- C4 pad 1: GNDPWR -> GND
- C4 pad 2: 3.3V -> +5V
- C5 pad 1: GND -> +12V
- C5 pad 2: +3V3 -> GNDPWR
- C6 pad 1: GND -> GNDPWR
- C6 pad 2: +5V -> 3.3V
- C7 pad 1: VCC -> 3.3V
- C8 pad 1: +12V -> VCC
- D10 pad 2: Solenoid_B1 -> Solenoid_B3
- D11 pad 2: Solenoid_B2 -> Solenoid_B4
- D12 pad 2: Solenoid_B3 -> Solenoid_A5
- D13 pad 2: Solenoid_B4 -> Solenoid_A6
- D14 pad 2: Solenoid_A5 -> Solenoid_A7
- D15 pad 2: Solenoid_A6 -> Solenoid_B5
- D16 pad 2: Solenoid_A7 -> Solenoid_B6
- D17 pad 2: Solenoid_B5 -> Solenoid_B7
- D2 pad 2: Solenoid_C1 -> Solenoid_C2
- D3 pad 2: Solenoid_C2 -> Solenoid_C3
- D4 pad 2: Solenoid_C3 -> Solenoid_A1
- D6 pad 2: Solenoid_A1 -> Solenoid_A3
- D7 pad 2: Solenoid_A2 -> Solenoid_A4
- D8 pad 2: Solenoid_A3 -> Solenoid_B1
- D9 pad 2: Solenoid_A4 -> Solenoid_B2
- J2 pad 1: 3.3V -> +12V
- J2 pad 2: /SWCLK -> Solenoid_C1
- J3 pad 2: Solenoid_A2 -> Solenoid_C2
- J4 pad 1: +12V -> GNDPWR
- J4 pad 2: Solenoid_C1 -> VCP_TX
- J5 pad 1: +12V -> 3.3V
- J5 pad 2: Solenoid_C2 -> /SWCLK
- J7 pad 1: GNDPWR -> +12V
- J7 pad 2: VCP_TX -> Solenoid_A1
- J8 pad 2: Solenoid_A1 -> Solenoid_A2
- Q3 pad 10: (no net) -> Net-(Q3-Pad10) (x2)
- Q3 pad 11: (no net) -> Net-(Q3-Pad11) (x2)
- Q3 pad 12: (no net) -> Net-(Q3-Pad12) (x2)
- Q3 pad 13: (no net) -> Net-(Q3-Pad13) (x2)
- Q3 pad 4: (no net) -> Net-(Q3-Pad4) (x2)
- Q3 pad 5: (no net) -> Net-(Q3-Pad5) (x2)
- Q3 pad 6: (no net) -> Net-(Q3-Pad6) (x2)
- Q3 pad 7: (no net) -> Net-(Q3-Pad7) (x2)
- R1 pad 2: +3V3 -> GNDPWR
- S1 pad 1: (no net) -> Net-(S1-Pad1) (x2)
- S1 pad 2: (no net) -> Net-(S1-Pad2) (x2)
- U2 pad 1: 3.3V -> CAN_TXD
- U2 pad 2: IC_B7 -> GND
- U2 pad 3: IC_B6 -> +5V
- U2 pad 4: NRST -> CAN_RXD
- U2 pad 5: 3.3V -> +3V3
- U2 pad 6: IC_B5 -> CAN-
- U2 pad 7: IC_B4 -> CAN+
- U2 pad 8: VCP_TX -> GND
- U3 pad 1: CAN_TXD -> 3.3V
- U3 pad 2: GND -> IC_B7
- U3 pad 3: +5V -> IC_B6
- U3 pad 4: CAN_RXD -> NRST
- U3 pad 5: +3V3 -> 3.3V
- U3 pad 6: CAN- -> IC_B5
- U3 pad 7: CAN+ -> IC_B4
- U3 pad 8: GND -> VCP_TX
- U4 pad 1: VCC -> GNDPWR
- U4 pad 2: GNDPWR -> 3.3V
- U5 pad 1: GNDPWR -> VCC
- U5 pad 2: 3.3V -> GNDPWR
Routing:
- net +12V: track 733.2 -> 627.9 mm
- net +3V3: track 164.7 -> 90.8 mm
- net IC_B1: track 94.8 -> 34.2 mm, vias 0 -> 4
- net IC_B3: track 83.3 -> 29.2 mm, vias 0 -> 4
- net +5V: track 117.1 -> 92.9 mm
- net NRST: track 40.6 -> 20.2 mm, vias 0 -> 2
- net VCC: track 90.8 -> 110.6 mm
- net /SWDIO: track 47.6 -> 30.8 mm
- net GND: track 54.3 -> 43.2 mm, vias 28 -> 32
- net VCP_TX: track 36.0 -> 45.5 mm
- net 3.3V: track 168.2 -> 177.6 mm
- net Net-(J1-PadB5): track 11.2 -> 2.00 mm
- net Net-(J1-PadA5): track 11.2 -> 2.00 mm
- net Net-(D1-Pad2): track 6.21 -> 0.00 mm
- net /BOOT: track 17.7 -> 11.5 mm, vias 4 -> 0
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Other:
- board size 85.9 x 100 mm -> 85.8 x 82.1 mm
